File: hardware/mainboard/isspointer/isspointer.sch (KiCad schematic (older format))
At the start: 24 parts, among them J1 USB_B_Micro, Q1 Q_NPN_BCE, Q2 Q_NPN_BCE, U1 AMS1117-3.3, U2 CP2102N-A01-GQFN28, U3 esp32-WROOM-32D

Commit message: esp32 pcb done
Parts:
- removed C2: C, symbol Device:C
- removed R7, R9: R_US, symbol Device:R_US
- added C1: 4.7uF/6.3V(10%), Capacitor_SMD:C_0603_1608Metric_Pad1.05x0.95mm_HandSolder, symbol Device:C
- added C4, C5: 22uF/10V(20%), Capacitor_SMD:C_0603_1608Metric_Pad1.05x0.95mm_HandSolder, symbol Device:C
- added C6, C7, C8, C9: 0.1uF/50V(10%), Capacitor_SMD:C_0603_1608Metric_Pad1.05x0.95mm_HandSolder, symbol Device:C
- added R2, R3: 0R(5%), Resistor_SMD:R_0603_1608Metric_Pad1.05x0.95mm_HandSolder, symbol Device:R_US
- added SW1, SW2: SW_Push, Button_Switch_SMD:SW_SPST_B3S-1000, symbol Switch:SW_Push
- added U4: DRV8834_HTSSOP, isspointer:DRV8834PWPR, symbol isspointer:DRV8834_HTSSOP
- C2: renamed from C1; value C -> 22uF/10V(20%); footprint (none) -> Capacitor_SMD:C_0603_1608Metric_Pad1.05x0.95mm_HandSolder
- C3: value C -> 0.1uF/50V(10%); footprint (none) -> Capacitor_SMD:C_0603_1608Metric_Pad1.05x0.95mm_HandSolder
- D1: footprint (none) -> Diode_SMD:D_0603_1608Metric
- D2: value D_TVS -> LESD5D5.0CT1G
- D3, D4: value D_TVS -> LESD5D5.0CT1G; footprint (none) -> Diode_SMD:D_SOD-523
- Q1, Q2: value Q_NPN_BCE -> SS8050-G; footprint (none) -> Package_TO_SOT_SMD:SOT-23
- R1: value R_US -> 2K(5%); footprint (none) -> Resistor_SMD:R_0603_1608Metric_Pad1.05x0.95mm_HandSolder
- R10: value R_US -> 10K(5%); footprint (none) -> Resistor_SMD:R_0603_1608Metric_Pad1.05x0.95mm_HandSolder
- R4: renamed from R6; value R_US -> 2K(5%); footprint (none) -> Resistor_SMD:R_0603_1608Metric_Pad1.05x0.95mm_HandSolder
- R5: renamed from R2; value R_US -> 22.1K(5%); footprint (none) -> Resistor_SMD:R_0603_1608Metric_Pad1.05x0.95mm_HandSolder
- R6: renamed from R5; value R_US -> 47.5K(5%); footprint (none) -> Resistor_SMD:R_0603_1608Metric_Pad1.05x0.95mm_HandSolder
- R7: renamed from R8; value R_US -> 10K(5%); footprint (none) -> Resistor_SMD:R_0603_1608Metric_Pad1.05x0.95mm_HandSolder
- R8: renamed from R4; value R_US -> 10K(5%); footprint (none) -> Resistor_SMD:R_0603_1608Metric_Pad1.05x0.95mm_HandSolder
- R9: renamed from R3; value R_US -> 10K(5%); footprint (none) -> Resistor_SMD:R_0603_1608Metric_Pad1.05x0.95mm_HandSolder
Connections:
- net labels added: CTS, DCD, DSR, DTR, EN, IO0, IO10, IO11, IO12, IO14, IO15, IO16, IO17, IO18, IO19, IO2, IO21, IO22, IO23, IO25, IO26, IO27, IO32, IO33, IO34, IO35, IO36, IO39, IO4, IO5, IO6, IO7, IO8, IO9, RI, RTS, RXD, RXD0, TXD, TXD0
- wire segments 50 -> 130
- no-connect marks 1 -> 12
Other:
- moved on the sheet: C2, D1, D2, D3, D4, D5, J1, Q1, R1, R4, R5, R6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

Commit message: stepper drivers
Parts:
- added C10, C17: 10nF/50V(10%), Capacitor_SMD:C_0603_1608Metric_Pad1.05x0.95mm_HandSolder, symbol Device:C
- added C11, C18: 4.7uF/6.3V(10%), Capacitor_SMD:C_0603_1608Metric_Pad1.05x0.95mm_HandSolder, symbol Device:C
- added C12, C19: 100 uF 16V, Capacitor_SMD:CP_Elec_6.3x4.9, symbol Device:CP1
- added C13, C16, C20, C23: 10uF/10V(20%), Capacitor_SMD:C_0603_1608Metric_Pad1.05x0.95mm_HandSolder, symbol Device:C
- added C14, C15, C21, C22: 0.1uF/50V(10%), Capacitor_SMD:C_0603_1608Metric_Pad1.05x0.95mm_HandSolder, symbol Device:C
- added J2: Motor 1, Connector_JST:JST_XH_B5B-XH-A_1x05_P2.50mm_Vertical, symbol Connector_Generic:Conn_01x05
- added J3: Motor 2, Connector_JST:JST_XH_B5B-XH-A_1x05_P2.50mm_Vertical, symbol Connector_Generic:Conn_01x05
- added R11, R14, R15, R19, R22, R23: 47K(5%), Resistor_SMD:R_0603_1608Metric_Pad1.05x0.95mm_HandSolder, symbol Device:R_US
- added R12, R20: 1.5K(5%), Resistor_SMD:R_0603_1608Metric_Pad1.05x0.95mm_HandSolder, symbol Device:R_US
- added R13, R21: 10K(5%), Resistor_SMD:R_0603_1608Metric_Pad1.05x0.95mm_HandSolder, symbol Device:R_US
- added R16, R17, R24, R25: 100(5%) 1W, Resistor_SMD:R_2512_6332Metric_Pad1.52x3.35mm_HandSolder, symbol Device:R_US
- added R18, R26: 1(20%), Resistor_SMD:R_0603_1608Metric_Pad1.05x0.95mm_HandSolder, symbol Device:R_US
- added RV1, RV2: R_POT_US, digikey-footprints:Trimpot_3.8mmx3.6mm_TC33X-2-103E, symbol Device:R_POT_US
- added U5: DRV8834_HTSSOP, isspointer:DRV8834PWPR, symbol isspointer:DRV8834_HTSSOP
- C2, C4, C5: footprint Capacitor_SMD:C_0603_1608Metric_Pad1.05x0.95mm_HandSolder -> Capacitor_SMD:C_1206_3216Metric_Pad1.42x1.75mm_HandSolder
Connections:
- net labels added: +3.3V, A1_1, A1_2, A2_1, A2_2, B1_1, B1_2, B2_1, B2_2, DIR_1, DIR_2, ENABLE_1, ENABLE_2, STEP_1, STEP_2
- net labels removed: VDD
- wire segments 130 -> 232
Other:
- note added: "ESP32"
- note added: "Motor 1"
- note added: "Motor 2"
- note added: "USB stuff"
- moved on the sheet: C1, C2, C3, C4, C5, C6, C7, C8, C9, D1, D2, D3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

Commit message: endstops and accel circuit board
Parts:
- added C24: 0.22uF/50V(10%), Capacitor_SMD:C_0603_1608Metric_Pad1.05x0.95mm_HandSolder, symbol Device:C
- added C25: 4.7uF/50V(10%), Capacitor_SMD:C_0603_1608Metric_Pad1.05x0.95mm_HandSolder, symbol Device:C
- added Q3, Q4: DMN67D8L, Package_TO_SOT_SMD:SOT-23, symbol Transistor_FET:DMN67D8L
- added R27, R28, R29, R30, R32, R34: 4.7K(5%), Resistor_SMD:R_0603_1608Metric_Pad1.05x0.95mm_HandSolder, symbol Device:R_US
- added R31, R33: 330(5%), Resistor_SMD:R_0603_1608Metric_Pad1.05x0.95mm_HandSolder, symbol Device:R_US
- added U6: LSM303DLHC, Package_LGA:LGA-14_3x5mm_P0.8mm_LayoutBorder1x6y, symbol Sensor_Motion:LSM303DLHC
- added U7, U8: EE-SX3350, isspointer:EE-SX3350, symbol isspointer:EE-SX3350
- C10, C17, C20: footprint Capacitor_SMD:C_0603_1608Metric_Pad1.05x0.95mm_HandSolder -> Capacitor_SMD:C_0402_1005Metric
- C11, C18: value 4.7uF/6.3V(10%) -> 2.2uF/6.3V(10%); footprint Capacitor_SMD:C_0603_1608Metric_Pad1.05x0.95mm_HandSolder -> Capacitor_SMD:C_0402_1005Metric
- C14: value 0.1uF/50V(10%) -> 10nF/50V(10%); footprint Capacitor_SMD:C_0603_1608Metric_Pad1.05x0.95mm_HandSolder -> Capacitor_SMD:C_0402_1005Metric
Connections:
- net ENABLE_2 is gone; now on net ENABLE_1: R21.2, U5.1 (~SLEEP)
- net IO14 is gone; now on net ENABLE_1: U3.13 (GPIO14)
- net IO26 is gone; now on net DIR_1: U3.11 (GPIO26)
- net IO27 is gone; now on net DIR_2: U3.12 (GPIO27)
- net STEP_1 is gone; now on net IO33: U4.11 (STEP/BENBL)
- net STEP_2 is gone; now on net IO25: U5.11 (STEP/BENBL)
- net +3V3: now also Q3.1 (G), Q4.1 (G), R27.1, R28.1, U6.1 (VDDIO), U6.14 (VDD)
- net +5V: now also R29.1, R30.1, R31.2, R32.1, R33.2, R34.1, U7.6, U8.6
- net GNDREF: now also RV1.3, RV2.3, U4.21 (GND), U4.25 (GNDpad), U5.21 (GND), U5.25 (GNDpad), C25.2, U6.10 (GND), U6.11 (GND), U6.7 (GND), U7.3, U7.4, U8.3, U8.4
- net IO21: now also Q4.3 (D), R30.2
- net IO22: now also Q3.3 (D), R29.2
- net ADECAY_1: now reaches R15.1, U4.3 (ADECAY)
- net AISEN_1: now reaches R17.1, U4.5 (AISEN)
- net BISEN_1: now reaches R16.2, U4.8 (BISEN)
- net BDECAY_1: now reaches R14.2, U4.2 (BDECAY)
- net nFAULT_1: now reaches R12.1, U4.16 (~FAULT)
- net CONFIG_1: now reaches R11.2, U4.15 (CONFIG)
- net VREF1: now reaches RV1.1, U4.24 (VREFO)
- net AVREF1: now reaches RV1.2, U4.22 (AVREF), U4.23 (BVREF)
- net IO36 renamed END_1
- net END_1: now also R32.2, U7.5
- net IO39 renamed END_2
- net END_2: now also R34.2, U8.5
- new net: C24.2, U6.12 (SETP)
- new net: C24.1, U6.13 (SETC)
- new net: C25.1, U6.6 (C1)
- new net: R31.1, U7.1
- new net: R33.1, U8.1
- new net DRDY: U6.9 (DRDY)
- new net INT1: U6.5 (INT1)
- new net INT2: U6.4 (INT2)
- new net SCLLV: Q3.2 (S), R27.2, U6.2 (SCL)
- new net SDALV: Q4.2 (S), R28.2, U6.3 (SDA)
Other:
- note added: "Accelerometer"
- note added: "Compass"
- note added: "Endstops"
- moved on the sheet: C5, C6, C7, R10

Commit message: display!
Parts:
- added C? (x4): 1.0uF/10V(10%), Capacitor_SMD:C_0603_1608Metric_Pad1.05x0.95mm_HandSolder, symbol Device:C
- added C? (x3): 2.2uF/10V(10%), Capacitor_SMD:C_0603_1608Metric_Pad1.05x0.95mm_HandSolder, symbol Device:C
- added R?: 300K(5%), Resistor_SMD:R_0603_1608Metric_Pad1.05x0.95mm_HandSolder, symbol Device:R_US
- added R?: 10K(5%), Resistor_SMD:R_0603_1608Metric_Pad1.05x0.95mm_HandSolder, symbol Device:R_US
- added U?: CFAL12864N, symbol isspointer:CFAL12864N
Connections:
- net +3V3: now also C?.2, R?.2, U?.11 (BS1), U?.6 (Vbat)
- net GNDREF: now also C?.1, R?.1, R?.1, U?.1 (GND), U?.10 (BS0), U?.12 (BS2), U?.29 (VLSS), U?.30 (GND), U?.8 (Vss(GND))
- new net: C?.1, U?.2 (C2N)
- new net: C?.2, U?.3 (C2P)
- new net: R?.2, U?.26 (Iref)
- new net: C?.1, U?.5 (C1N)
- new net: C?.2, U?.4 (C1P)
Other:
- note added: "Display"

Commit message: gps
Parts:
- removed C? (x3): 1.0uF/10V(10%), Capacitor_SMD:C_0603_1608Metric_Pad1.05x0.95mm_HandSolder, symbol Device:C
- added C27: 2.2uF/16V(10%), Capacitor_SMD:C_0603_1608Metric_Pad1.05x0.95mm_HandSolder, symbol Device:C
- added C28: 2.2uF/10V(10%), Capacitor_SMD:C_0603_1608Metric_Pad1.05x0.95mm_HandSolder, symbol Device:C
- added C?: 0.1uF/50V(10%), Capacitor_SMD:C_0603_1608Metric_Pad1.05x0.95mm_HandSolder, symbol Device:C
- added D?: LED, Diode_SMD:D_0603_1608Metric, symbol Device:LED
- added J?: U_FL-R-SMT-1_10_, digikey-footprints:Coax_Conn_U.FL, symbol dk_Coaxial-Connectors-RF:U_FL-R-SMT-1_10_
- added R35, R36, R37, R?: 10K(5%), Resistor_SMD:R_0603_1608Metric_Pad1.05x0.95mm_HandSolder, symbol Device:R_US
- added R?: 1K(5%), Resistor_SMD:R_0603_1608Metric_Pad1.05x0.95mm_HandSolder, symbol Device:R_US
- added SW3: Up, Button_Switch_THT:SW_TH_Tactile_Omron_B3F-10xx, symbol Switch:SW_Push
- added SW4: Select, Button_Switch_THT:SW_TH_Tactile_Omron_B3F-10xx, symbol Switch:SW_Push
- added SW5: Down, Button_Switch_THT:SW_TH_Tactile_Omron_B3F-10xx, symbol Switch:SW_Push
- added U?: TPS79133-EP, Package_TO_SOT_SMD:SOT-23-6, symbol isspointer:TPS79133-EP
- added U?: NEO-6M-0-001, RF_GPS:ublox_NEO, symbol isspointer:NEO-6M-0-001
- added U?: 24AA32-OT, Package_SO:SOIC-8_3.9x4.9mm_P1.27mm, symbol isspointer:24AA32-OT
- C30: renamed from C?; value 1.0uF/10V(10%) -> 10uF/10V(10%)
- SW1: value SW_Push -> Boot; footprint Button_Switch_SMD:SW_SPST_B3S-1000 -> Button_Switch_SMD:SW_SPST_CK_RS282G05A3
- SW2: value SW_Push -> Reset; footprint Button_Switch_SMD:SW_SPST_B3S-1000 -> Button_Switch_SMD:SW_SPST_CK_RS282G05A3
- U9: renamed from U?; footprint (none) -> isspointer:CFAL12864N_oled
- gave numbers to parts that had none: 5
Connections:
- net +3V3: now also U9.9 (Vlogic), C28.1, C?.1, SW3.1, SW4.1, SW5.1, U?.23 (VCC), U?.8 (VCC)
- net GNDREF: now also C30.1, R38.2, U9.15 (D/C#_SA0), C27.1, C28.2, C?.2, D?.1 (K), R35.1, R36.1, R37.1, U?.1 (A0), U?.2 (A1), U?.3 (A2), U?.4 (GND), U?.7 (WP); no longer R38.1
- net SCLLV: now also U9.18 (D0_SCL)
- net SDALV: now also U9.19 (D1_SDAin), U9.20 (D2_SDAout)
- net at U9.26 (Iref): now also R38.1; no longer R38.2
- net at C30.2: now also U9.28 (Voled)
- net at U9.27 (Vcomh): now also C27.2
- net IO32 renamed BTN_DOWN
- net BTN_DOWN: now also R37.2, SW5.2
- net IO34 renamed BTN_UP
- net BTN_UP: now also R35.2, SW3.2
- net IO35 renamed BTN_SELECT
- net BTN_SELECT: now also R36.2, SW4.2
- new net: U?.10 (GND), U?.12 (GND), U?.13 (GND), U?.24 (GND)
- new net: R?.2, U?.3 (TIMEPULSE)
- new net: D?.2 (A), R?.1
- new net SCL2: U?.19 (SCL2), U?.6 (SCL)
- new net SDA2: U?.18 (SDA2), U?.5 (SDA)
Other:
- note added: "Buttons"
- note added: "GPS"
- note added: "address 0x78 with SA0 at GND"
- moved on the sheet: C26, C29, C30, C31, R38, R39, U9

Commit message: 3v battery
Parts:
- added BT?: 3V lithium cell, isspointer:MS412FE_FL26E, symbol Device:Battery_Cell
Changed lines of the file:
@@
 Wire Wire Line
 	12400 12100 12400 12200
+$Comp
+L Device:Battery_Cell BT?
+U 1 1 5E58378E
+P 13400 12050
+F 0 "BT?" H 13518 12146 50  0000 L CNN
+F 1 "3V lithium cell" H 13518 12055 50  0000 L CNN
+F 2 "isspointer:MS412FE_FL26E" V 13400 12110 50  0001 C CNN
+F 3 "~" V 13400 12110 50  0001 C CNN
+	1    13400 12050
+	1    0    0    -1
+$EndComp
 $EndSCHEMATC

Commit message: minor
Parts:
- added L?: 27 uH MLF2012C270KT000, symbol isspointer-eagle-import:INDUCTOR0805
- added R?: 22(5%), Resistor_SMD:R_0603_1608Metric_Pad1.05x0.95mm_HandSolder, symbol Device:R_US
Connections:
- net GNDREF: now also J?.1
- net at J?.2: now also L?.1
- new net: L?.2, R?.1
Other:
- moved on the sheet: D?, J?, R?, U?
Changed lines of the file:
@@
 L isspointer:NEO-6M-0-001 U?
 U 1 1 5E5771B3
-P 10650 11800
-F 0 "U?" H 10650 10811 50  0000 C CNN
-F 1 "NEO-6M-0-001" H 10650 10720 50  0000 C CNN
-F 2 "RF_GPS:ublox_NEO" H 11050 10950 50  0001 C CNN
-F 3 "https://www.u-blox.com/sites/default/files/NEO-M8-FW3_DataSheet_%28UBX-15031086%29.pdf" H 10650 11800 50  0001 C CNN
-	1    10650 11800
+P 10000 12100
+F 0 "U?" H 10000 11111 50  0000 C CNN
+F 1 "NEO-6M-0-001" H 10000 11020 50  0000 C CNN
+F 2 "RF_GPS:ublox_NEO" H 10400 11250 50  0001 C CNN
+F 3 "https://www.u-blox.com/sites/default/files/NEO-M8-FW3_DataSheet_%28UBX-15031086%29.pdf" H 10000 12100 50  0001 C CNN
+	1    10000 12100
 	1    0    0    -1
 $EndComp
@@
 L isspointer:TPS79133-EP U?
 U 1 1 5E552781
-P 8950 12400
-F 0 "U?" H 8950 12742 50  0000 C CNN
-F 1 "TPS79133-EP" H 8950 12651 50  0000 C CNN
-F 2 "Package_TO_SOT_SMD:SOT-23-6" H 8950 12725 50  0001 C CIN
-F 3 "http://www.ti.com/lit/ds/symlink/tps79333-ep.pdf" H 8950 12450 50  0001 C CNN
-	1    8950 12400
+P 8300 12700
+F 0 "U?" H 8300 13042 50  0000 C CNN
+F 1 "TPS79133-EP" H 8300 12951 50  0000 C CNN
+F 2 "Package_TO_SOT_SMD:SOT-23-6" H 8300 13025 50  0001 C CIN
+F 3 "http://www.ti.com/lit/ds/symlink/tps79333-ep.pdf" H 8300 12750 50  0001 C CNN
+	1    8300 12700
 	1    0    0    -1
 $EndComp
@@
 	1    0    0    -1
 $EndComp
-Text Label 9700 11800 0    50   ~ 0
+Text Label 9050 12100 0    50   ~ 0
 SDA2
-Text Label 9700 11900 0    50   ~ 0
+Text Label 9050 12200 0    50   ~ 0
 SCL2
 Wire Wire Line
-	9950 11800 9700 11800
-Wire Wire Line
-	9950 11900 9700 11900
+	9300 12100 9050 12100
+Wire Wire Line
+	9300 12200 9050 12200
 Text Label 13700 10700 2    50   ~ 0
 SDA2
@@
 L dk_Coaxial-Connectors-RF:U_FL-R-SMT-1_10_ J?
 U 1 1 5E7CAB51
-P 9100 10950
-F 0 "J?" H 9178 11175 50  0000 C CNN
-F 1 "U_FL-R-SMT-1_10_" H 9178 11084 50  0000 C CNN
-F 2 "digikey-footprints:Coax_Conn_U.FL" H 9300 11150 60  0001 L CNN
-F 3 "https://www.hirose.com/product/en/download_file/key_name/U.FL-R-SMT-1%2810%29/category/Drawing%20(2D)/doc_file_id/37627/?file_category_id=6&item_id=03310472210&is_series=U.FL-R-SMT-1(10" H 9300 11250 60  0001 L CNN
-F 4 "H11891CT-ND" H 9300 11350 60  0001 L CNN "Digi-Key_PN"
-F 5 "U.FL-R-SMT-1(10)" H 9300 11450 60  0001 L CNN "MPN"
-F 6 "Connectors, Interconnects" H 9300 11550 60  0001 L CNN "Category"
-F 7 "Coaxial Connectors (RF)" H 9300 11650 60  0001 L CNN "Family"
-F 8 "https://www.hirose.com/product/en/download_file/key_name/U.FL-R-SMT-1%2810%29/category/Drawing%20(2D)/doc_file_id/37627/?file_category_id=6&item_id=03310472210&is_series=U.FL-R-SMT-1(10" H 9300 11750 60  0001 L CNN "DK_Datasheet_Link"
-F 9 "/product-detail/en/hirose-electric-co-ltd/U.FL-R-SMT-1(10)/H11891CT-ND/2504612" H 9300 11850 60  0001 L CNN "DK_Detail_Page"
-F 10 "CONN U.FL RCPT STR 50 OHM SMD" H 9300 11950 60  0001 L CNN "Description"
-F 11 "Hirose Electric Co Ltd" H 9300 12050 60  0001 L CNN "Manufacturer"
-F 12 "Active" H 9300 12150 60  0001 L CNN "Status"
-	1    9100 10950
+P 11250 10550
+F 0 "J?" H 11328 10775 50  0000 C CNN
+F 1 "U_FL-R-SMT-1_10_" H 11328 10684 50  0000 C CNN
+F 2 "digikey-footprints:Coax_Conn_U.FL" H 11450 10750 60  0001 L CNN
+F 3 "https://www.hirose.com/product/en/download_file/key_name/U.FL-R-SMT-1%2810%29/category/Drawing%20(2D)/doc_file_id/37627/?file_category_id=6&item_id=03310472210&is_series=U.FL-R-SMT-1(10" H 11450 10850 60  0001 L CNN
+F 4 "H11891CT-ND" H 11450 10950 60  0001 L CNN "Digi-Key_PN"
+F 5 "U.FL-R-SMT-1(10)" H 11450 11050 60  0001 L CNN "MPN"
+F 6 "Connectors, Interconnects" H 11450 11150 60  0001 L CNN "Category"
+F 7 "Coaxial Connectors (RF)" H 11450 11250 60  0001 L CNN "Family"
+F 8 "https://www.hirose.com/product/en/download_file/key_name/U.FL-R-SMT-1%2810%29/category/Drawing%20(2D)/doc_file_id/37627/?file_category_id=6&item_id=03310472210&is_series=U.FL-R-SMT-1(10" H 11450 11350 60  0001 L CNN "DK_Datasheet_Link"
+F 9 "/product-detail/en/hirose-electric-co-ltd/U.FL-R-SMT-1(10)/H11891CT-ND/2504612" H 11450 11450 60  0001 L CNN "DK_Detail_Page"
+F 10 "CONN U.FL RCPT STR 50 OHM SMD" H 11450 11550 60  0001 L CNN "Description"
+F 11 "Hirose Electric Co Ltd" H 11450 11650 60  0001 L CNN "Manufacturer"
+F 12 "Active" H 11450 11750 60  0001 L CNN "Status"
+	1    11250 10550
 	1    0    0    -1
 $EndComp
@@
 L Device:R_US R?
 U 1 1 5E7CC5CF
-P 9450 11950
-F 0 "R?" H 9382 11904 50  0000 R CNN
-F 1 "10K(5%)" H 9382 11995 50  0000 R CNN
-F 2 "Resistor_SMD:R_0603_1608Metric_Pad1.05x0.95mm_HandSolder" V 9490 11940 50  0001 C CNN
-F 3 "~" H 9450 11950 50  0001 C CNN
-	1    9450 11950
+P 8800 12250
+F 0 "R?" H 8732 12204 50  0000 R CNN
+F 1 "10K(5%)" H 8732 12295 50  0000 R CNN
+F 2 "Resistor_SMD:R_0603_1608Metric_Pad1.05x0.95mm_HandSolder" V 8840 12240 50  0001 C CNN
+F 3 "~" H 8800 12250 50  0001 C CNN
+	1    8800 12250
 	0    1    1    0
 $EndComp
@@
 L power:+3.3V #PWR?
 U 1 1 5E7F5B7C
-P 10250 10700
-F 0 "#PWR?" H 10250 10550 50  0001 C CNN
-F 1 "+3.3V" H 10267 10873 50  0000 C CNN
-F 2 "" H 10250 10700 50  0001 C CNN
-F 3 "" H 10250 10700 50  0001 C CNN
-	1    10250 10700
-	1    0    0    -1
-$EndComp
-Wire Wire Line
-	10450 10900 10450 10800
-Wire Wire Line
-	10450 10800 10250 10800
-Wire Wire Line
-	10250 10800 10250 10700
+P 9600 11000
+F 0 "#PWR?" H 9600 10850 50  0001 C CNN
+F 1 "+3.3V" H 9617 11173 50  0000 C CNN
+F 2 "" H 9600 11000 50  0001 C CNN
+F 3 "" H 9600 11000 50  0001 C CNN
+	1    9600 11000
+	1    0    0    -1
+$EndComp
+Wire Wire Line
+	9800 11200 9800 11100
+Wire Wire Line
+	9800 11100 9600 11100
+Wire Wire Line
+	9600 11100 9600 11000
 $Comp
 L Device:R_US R?
 U 1 1 5E81CF2E
-P 11650 12100
-F 0 "R?" H 11582 12054 50  0000 R CNN
-F 1 "1K(5%)" H 11582 12145 50  0000 R CNN
-F 2 "Resistor_SMD:R_0603_1608Metric_Pad1.05x0.95mm_HandSolder" V 11690 12090 50  0001 C CNN
-F 3 "~" H 11650 12100 50  0001 C CNN
-	1    11650 12100
+P 11000 12400
+F 0 "R?" H 10932 12354 50  0000 R CNN
+F 1 "1K(5%)" H 10932 12445 50  0000 R CNN
+F 2 "Resistor_SMD:R_0603_1608Metric_Pad1.05x0.95mm_HandSolder" V 11040 12390 50  0001 C CNN
+F 3 "~" H 11000 12400 50  0001 C CNN
+	1    11000 12400
 	0    1    1    0
 $EndComp
@@
 L Device:LED D?
 U 1 1 5E81DA44
-P 12100 12100
-F 0 "D?" V 12139 11983 50  0000 R CNN
-F 1 "LED" V 12048 11983 50  0000 R CNN
-F 2 "Diode_SMD:D_0603_1608Metric" H 12100 12100 50  0001 C CNN
-F 3 "~" H 12100 12100 50  0001 C CNN
-	1    12100 12100
+P 11450 12400
+F 0 "D?" V 11489 12283 50  0000 R CNN
+F 1 "LED" V 11398 12283 50  0000 R CNN
+F 2 "Diode_SMD:D_0603_1608Metric" H 11450 12400 50  0001 C CNN
+F 3 "~" H 11450 12400 50  0001 C CNN
+	1    11450 12400
 	-1   0    0    1
 $EndComp
@@
 L power:GNDREF #PWR?
 U 1 1 5E81F476
-P 12400 12200
-F 0 "#PWR?" H 12400 11950 50  0001 C CNN
-F 1 "GNDREF" H 12405 12027 50  0001 C CNN
-F 2 "" H 12400 12200 50  0001 C CNN
-F 3 "" H 12400 12200 50  0001 C CNN
-	1    12400 12200
-	1    0    0    -1
-$EndComp
-Wire Wire Line
-	11350 12100 11500 12100
-Wire Wire Line
-	11800 12100 11950 12100
-Wire Wire Line
-	12250 12100 12400 12100
-Wire Wire Line
-	12400 12100 12400 12200
+P 11750 12500
+F 0 "#PWR?" H 11750 12250 50  0001 C CNN
+F 1 "GNDREF" H 11755 12327 50  0001 C CNN
+F 2 "" H 11750 12500 50  0001 C CNN
+F 3 "" H 11750 12500 50  0001 C CNN
+	1    11750 12500
+	1    0    0    -1
+$EndComp
+Wire Wire Line
+	10700 12400 10850 12400
+Wire Wire Line
+	11150 12400 11300 12400
+Wire Wire Line
+	11600 12400 11750 12400
+Wire Wire Line
+	11750 12400 11750 12500
 $Comp
 L Device:Battery_Cell BT?
@@
 	1    0    0    -1
 $EndComp
+$Comp
+L isspointer-eagle-import:INDUCTOR0805 L?
+U 1 1 5E55D339
+P 11200 11200
+F 0 "L?" V 10998 11200 59  0000 C CNN
+F 1 "27 uH MLF2012C270KT000 " V 11103 11200 59  0000 C CNN
+F 2 "" H 11200 11200 50  0001 C CNN
+F 3 "" H 11200 11200 50  0001 C CNN
+	1    11200 11200
+	0    1    1    0
+$EndComp
+$Comp
+L Device:R_US R?
+U 1 1 5E55ED90
+P 10550 11200
+F 0 "R?" H 10482 11154 50  0000 R CNN
+F 1 "22(5%)" H 10482 11245 50  0000 R CNN
+F 2 "Resistor_SMD:R_0603_1608Metric_Pad1.05x0.95mm_HandSolder" V 10590 11190 50  0001 C CNN
+F 3 "~" H 10550 11200 50  0001 C CNN
+	1    10550 11200
+	0    1    1    0
+$EndComp
+Wire Wire Line
+	10200 11200 10400 11200
+Wire Wire Line
+	10700 11200 10900 11200
+Wire Wire Line
+	11500 11200 11500 10550
+Wire Wire Line
+	11500 10550 11450 10550
+$Comp
+L power:GNDREF #PWR?
+U 1 1 5E60C9CA
+P 11250 10750
+F 0 "#PWR?" H 11250 10500 50  0001 C CNN
+F 1 "GNDREF" H 11255 10577 50  0001 C CNN
+F 2 "" H 11250 10750 50  0001 C CNN
+F 3 "" H 11250 10750 50  0001 C CNN
+	1    11250 10750
+	1    0    0    -1
+$EndComp

Commit message: some trace routing
Parts:
- removed R?: 10K(5%), Resistor_SMD:R_0603_1608Metric_Pad1.05x0.95mm_HandSolder, symbol Device:R_US
- removed U?: TPS79133-EP, Package_TO_SOT_SMD:SOT-23-6, symbol isspointer:TPS79133-EP
- added C33: 4.7uF, Capacitor_SMD:C_0603_1608Metric_Pad1.05x0.95mm_HandSolder, symbol Device:C
- added D6: D_Schottky, Diode_SMD:D_SOD-323_HandSoldering, symbol Device:D_Schottky
- added R40: 1K(5%), Resistor_SMD:R_0603_1608Metric_Pad1.05x0.95mm_HandSolder, symbol Device:R_US
- L1: renamed from L?; footprint (none) -> Inductor_SMD:L_0805_2012Metric_Pad1.15x1.40mm_HandSolder
- RV1, RV2: value R_POT_US -> 10K TRIMMER
- SW3, SW4, SW5: footprint Button_Switch_THT:SW_TH_Tactile_Omron_B3F-10xx -> Button_Switch_SMD:SW_SPST_B3S-1000
- gave numbers to parts that had none: 8
Connections:
- net IO16 is gone; now on net ESP_RXD1: U3.27 (GPIO16)
- net IO17 is gone; now on net ESP_TXD1: U3.28 (GPIO17)
- net +3V3: now also C33.1, D6.2 (A)
- net GNDREF: now also BT1.2 (-), U10.10 (GND), U10.12 (GND), U10.13 (GND), U10.24 (GND), U10.7 (VDD_USB), C33.2
- net at J4.2, L1.1: now also U10.11 (RF_IN)
- net at L1.2: now also R42.2; no longer R42.1
- net ESP_RXD1: now reaches U10.20 (TXD1)
- net ESP_TXD1: now reaches U10.21 (RXD1)
- net at U10.22 (V_BCKP): now also BT1.1 (+), R40.2
- net VCC_RF: now reaches U10.8 (~RESET)
- net VCC_RF: now also R42.1, U10.9 (VCC_RF)
- net SCL2 renamed NEO_SCL2
- net SDA2 renamed NEO_SDA2
- new net: D6.1 (K), R40.1
Other:
- note added: "I2C EEPROM"
- note added: "\n\USB communication\n/"
- note added: "|\n|GPS communication\n|"
- moved on the sheet: BT1, C32, D7, J4, L1, R41, R42, U10, U11
