File: hardware/mainboard/isspointer/isspointer.sch (KiCad schematic (older format))
At the start: 110 parts, among them J1 USB_B_Micro, J2 Motor 1, J3 Motor 2, J4 U_FL-R-SMT-1_10_, Q1 SS8050-G, Q2 SS8050-G, Q3 DMN67D8L, Q4 DMN67D8L, SW1 Boot, SW2 Reset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

Commit message: working on perf board with endstops
Parts:
- added J?: Conn_01x04_Male, symbol Connector:Conn_01x04_Male
Connections:
- net +5V: now also J?.1 (Pin_1)
- net END_1: now also J?.2 (Pin_2)
- net END_2: now also J?.3 (Pin_3)
- net GNDREF: now also J?.4 (Pin_4)
Other:
- moved on the sheet: R31, R32, R33, R34, U7, U8
